File: Star-Notifier.kicad_pcb (KiCad board)
At the start: 2 copper layers, 45.1 x 43.2 mm, 40 parts, among them J1 HRO TYPE-C-31-M-12, SW1 RESET, SW2 BOOT, U1 USBLC6-2SC6, U2 AP2112K-3.3, U3 ESP32-C3-WROOM-02, U4 74AHCT1G125

Commit message: Move C1 next to F1 so its GND pad joins the main pour
C1's GND pad sat in a B.Cu pocket sealed off by the USB pair, leaving
an isolated pour island. It now sits beside F1's +5V pad with a short
0.6 mm link; DRC reports no unconnected items.

Co-Authored-By: Claude Opus 5.5 <noreply@anthropic.com>
Parts:
- moved C1 5.00 mm to (146.0, 113.3)
Routing:
- net +5V: track 138.9 -> 137.6 mm
Changed lines of the file:
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@@
 	(footprint "Capacitor_SMD:C_0805_2012Metric"
 		(layer "B.Cu")
-		(at 150 110.3 180)
+		(at 146 113.3 180)
 		(descr "Capacitor SMD 0805 (2012 Metric), square (rectangular) end terminal, IPC-7351 nominal, (Body size source: IPC-SM-782 page 76, https://www.pcb-3d.com/wordpress/wp-content/uploads/ipc-sm-782a_amendment_1_and_2.pdf, https://docs.google.com/spreadsheets/d/1BsfQQcO9C6DZCsRaXUlFlo91Tg2WpOkGARC1WS5S8t0/edit?usp=sharing)")
 		(tags "capacitor")
@@
 	)
 	(segment
-		(start 150.8537 111.742)
-		(end 150.8537 110.3963)
-		(width 0.4)
-		(layer "B.Cu")
-		(net "+5V")
-	)
-	(segment
 		(start 165.55 98.8421)
 		(end 165.55 100.6299)
@@
 	)
 	(segment
-		(start 149.7216 112.6717)
-		(end 149.924 112.6717)
-		(width 0.8)
-		(layer "B.Cu")
-		(net "+5V")
-	)
-	(segment
-		(start 150.8537 110.3963)
-		(end 150.95 110.3)
-		(width 0.6)
-		(layer "B.Cu")
-		(net "+5V")
-	)
-	(segment
 		(start 136.5699 98.0504)
 		(end 135.9695 97.45)
@@
 	)
 	(segment
-		(start 149.924 112.6717)
-		(end 150.8537 111.742)
-		(width 0.4)
+		(start 146.95 113.3)
+		(end 148.6 113.3)
+		(width 0.6)
 		(layer "B.Cu")
 		(net "+5V")
